Commit message: Change package name to walktoy

File: urdf/robot.xacro (robot description, xacro)
@@ -1,4 +1,5 @@
 <?xml version="1.0"?>
-<robot name="exoskeleton" xmlns:xacro="http://www.ros.org/wiki/xacro">
+<robot name="walktoy"
+  xmlns:xacro="http://www.ros.org/wiki/xacro">
   <xacro:property name="PI" value="3.1415926535897931"/>
   <!--waist property-->
@@ -35,10 +36,10 @@
   <xacro:property name="foot_maxvel" value="${PI}" />
   <!-- Import all Gazebo-customization elements, including Gazebo colors -->
-  <xacro:include filename="$(find exoskeleton)/urdf/robot.gazebo" />
+  <xacro:include filename="$(find walktoy)/urdf/robot.gazebo" />
   <link name="waist_link">
     <collision>
       <origin xyz="${-waist_height/2-up_width/2} 0 0" rpy="0 0 0"/>
       <geometry>
-	    <box size="${waist_height} ${waist_length} ${waist_width}"/>
+        <box size="${waist_height} ${waist_length} ${waist_width}"/>
       </geometry>
     </collision>
@@ -46,5 +47,5 @@
       <origin xyz="${-waist_height/2-up_width/2} 0 0" rpy="0 0 0"/>
       <geometry>
-	    <box size="${waist_height} ${waist_length} ${waist_width}"/>
+        <box size="${waist_height} ${waist_length} ${waist_width}"/>
       </geometry>
       <material name="orange"/>
@@ -53,13 +54,9 @@
       <origin xyz="${-waist_height/2-up_width/2} 0 0" rpy="0 0 0"/>
       <mass value="${waist_mass}"/>
-      <inertia
-	  ixx="${waist_mass / 12.0 * (waist_length*waist_length + waist_width*waist_width)}" ixy="0.0" ixz="0.0"
-	  iyy="${waist_mass / 12.0 * (waist_height*waist_height + waist_width*waist_width)}" iyz="0.0"
-	  izz="${waist_mass / 12.0 * (waist_height*waist_height + waist_length*waist_length)}"/>
+      <inertia ixx="${waist_mass / 12.0 * (waist_length*waist_length + waist_width*waist_width)}" ixy="0.0" ixz="0.0" iyy="${waist_mass / 12.0 * (waist_height*waist_height + waist_width*waist_width)}" iyz="0.0" izz="${waist_mass / 12.0 * (waist_height*waist_height + waist_length*waist_length)}"/>
     </inertial>
   </link>
   <joint name="LU_joint" type="revolute">
-    <limit
-        velocity="${up_maxvel}" effort="${up_effort}" lower="${up_lower}" upper="${up_upper}" />
+    <limit velocity="${up_maxvel}" effort="${up_effort}" lower="${up_lower}" upper="${up_upper}" />
     <parent link="waist_link"/>
     <child link="LU_link"/>
@@ -72,5 +69,5 @@
       <origin xyz="0 ${up_height/2} ${-(up_length/2)}" rpy="0 0 0"/>
       <geometry>
-	    <box size="${up_width} ${up_height} ${up_length}"/>
+        <box size="${up_width} ${up_height} ${up_length}"/>
       </geometry>
     </collision>
@@ -78,5 +75,5 @@
       <origin xyz="0 ${up_height/2} ${-(up_length/2)}" rpy="0 0 0"/>
       <geometry>
-	    <box size="${up_width} ${up_height} ${up_length}"/>
+        <box size="${up_width} ${up_height} ${up_length}"/>
       </geometry>
       <material name="orange"/>
@@ -85,13 +82,9 @@
       <origin xyz="0 ${up_height/2} ${-(up_length/2)}" rpy="0 0 0"/>
       <mass value="${up_mass}"/>
-      <inertia
-	  ixx="${up_mass / 12.0 * (up_height*up_height + up_length*up_length)}" ixy="0.0" ixz="0.0"
-	  iyy="${up_mass / 12.0 * (up_width*up_width + up_length*up_length)}" iyz="0.0"
-	  izz="${up_mass / 12.0 * (up_width*up_width + up_height*up_height)}"/>
+      <inertia ixx="${up_mass / 12.0 * (up_height*up_height + up_length*up_length)}" ixy="0.0" ixz="0.0" iyy="${up_mass / 12.0 * (up_width*up_width + up_length*up_length)}" iyz="0.0" izz="${up_mass / 12.0 * (up_width*up_width + up_height*up_height)}"/>
     </inertial>
   </link>
   <joint name="RU_joint" type="revolute">
-    <limit
-        velocity="${up_maxvel}"  effort="${up_effort}" lower="${up_lower}" upper="${up_upper}" />
+    <limit velocity="${up_maxvel}" effort="${up_effort}" lower="${up_lower}" upper="${up_upper}" />
     <parent link="waist_link"/>
     <child link="RU_link"/>
@@ -104,5 +97,5 @@
       <origin xyz="0 ${-up_height/2} ${-(up_length/2)}" rpy="0 0 0"/>
       <geometry>
-	    <box size="${up_width} ${up_height} ${up_length}"/>
+        <box size="${up_width} ${up_height} ${up_length}"/>
       </geometry>
     </collision>
@@ -110,5 +103,5 @@
       <origin xyz="0 ${-up_height/2} ${-(up_length/2)}" rpy="0 0 0"/>
       <geometry>
-	    <box size="${up_width} ${up_height} ${up_length}"/>
+        <box size="${up_width} ${up_height} ${up_length}"/>
       </geometry>
       <material name="orange"/>
@@ -117,13 +110,9 @@
       <origin xyz="0 ${-up_height/2} ${-(up_length/2)}" rpy="0 0 0"/>
       <mass value="${up_mass}"/>
-      <inertia
-	  ixx="${up_mass / 12.0 * (up_height*up_height + up_length*up_length)}" ixy="0.0" ixz="0.0"
-	  iyy="${up_mass / 12.0 * (up_width*up_width + up_length*up_length)}" iyz="0.0"
-	  izz="${up_mass / 12.0 * (up_width*up_width + up_height*up_height)}"/>
+      <inertia ixx="${up_mass / 12.0 * (up_height*up_height + up_length*up_length)}" ixy="0.0" ixz="0.0" iyy="${up_mass / 12.0 * (up_width*up_width + up_length*up_length)}" iyz="0.0" izz="${up_mass / 12.0 * (up_width*up_width + up_height*up_height)}"/>
     </inertial>
   </link>
   <joint name="LD_joint" type="revolute">
-    <limit
-        velocity="${down_maxvel}"  effort="${down_effort}" lower="${down_lower}" upper="${down_upper}" />
+    <limit velocity="${down_maxvel}" effort="${down_effort}" lower="${down_lower}" upper="${down_upper}" />
     <parent link="LU_link"/>
     <child link="LD_link"/>
@@ -136,5 +125,5 @@
       <origin xyz="0 ${-down_height/2} ${-(down_length/2)}" rpy="0 0 0"/>
       <geometry>
-	    <box size="${down_width} ${down_height} ${down_length}"/>
+        <box size="${down_width} ${down_height} ${down_length}"/>
       </geometry>
     </collision>
@@ -142,5 +131,5 @@
       <origin xyz="0 ${-down_height/2} ${-(down_length/2)}" rpy="0 0 0"/>
       <geometry>
-	    <box size="${down_width} ${down_height} ${down_length}"/>
+        <box size="${down_width} ${down_height} ${down_length}"/>
       </geometry>
       <material name="orange"/>
@@ -149,13 +138,9 @@
       <origin xyz="0 ${-down_height/2} ${-(down_length/2)}" rpy="0 0 0"/>
       <mass value="${down_mass}"/>
-      <inertia
-	  ixx="${down_mass / 12.0 * (down_height*down_height + down_length*down_length)}" ixy="0.0" ixz="0.0"
-	  iyy="${down_mass / 12.0 * (down_width*down_width + down_length*down_length)}" iyz="0.0"
-	  izz="${down_mass / 12.0 * (down_width*down_width + down_height*down_height)}"/>
+      <inertia ixx="${down_mass / 12.0 * (down_height*down_height + down_length*down_length)}" ixy="0.0" ixz="0.0" iyy="${down_mass / 12.0 * (down_width*down_width + down_length*down_length)}" iyz="0.0" izz="${down_mass / 12.0 * (down_width*down_width + down_height*down_height)}"/>
     </inertial>
   </link>
   <joint name="RD_joint" type="revolute">
-    <limit
-       velocity="${down_maxvel}" effort="${down_effort}" lower="${down_lower}" upper="${down_upper}" />
+    <limit velocity="${down_maxvel}" effort="${down_effort}" lower="${down_lower}" upper="${down_upper}" />
     <parent link="RU_link"/>
     <child link="RD_link"/>
@@ -168,5 +153,5 @@
       <origin xyz="0 ${down_height/2} ${-(down_length/2)}" rpy="0 0 0"/>
       <geometry>
-	    <box size="${down_width} ${down_height} ${down_length}"/>
+        <box size="${down_width} ${down_height} ${down_length}"/>
       </geometry>
     </collision>
@@ -174,5 +159,5 @@
       <origin xyz="0 ${down_height/2} ${-(down_length/2)}" rpy="0 0 0"/>
       <geometry>
-	    <box size="${down_width} ${down_height} ${down_length}"/>
+        <box size="${down_width} ${down_height} ${down_length}"/>
       </geometry>
       <material name="orange"/>
@@ -181,13 +166,9 @@
       <origin xyz="0 ${down_height/2} ${-(down_length/2)}" rpy="0 0 0"/>
       <mass value="${down_mass}"/>
-      <inertia
-	  ixx="${down_mass / 12.0 * (down_height*down_height + down_length*down_length)}" ixy="0.0" ixz="0.0"
-	  iyy="${down_mass / 12.0 * (down_width*down_width + down_length*down_length)}" iyz="0.0"
-	  izz="${down_mass / 12.0 * (down_width*down_width + down_height*down_height)}"/>
+      <inertia ixx="${down_mass / 12.0 * (down_height*down_height + down_length*down_length)}" ixy="0.0" ixz="0.0" iyy="${down_mass / 12.0 * (down_width*down_width + down_length*down_length)}" iyz="0.0" izz="${down_mass / 12.0 * (down_width*down_width + down_height*down_height)}"/>
     </inertial>
   </link>
   <joint name="LF_joint" type="revolute">
-    <limit
-       velocity="${foot_maxvel}" effort="${foot_effort}" lower="${foot_lower}" upper="${foot_upper}" />
+    <limit velocity="${foot_maxvel}" effort="${foot_effort}" lower="${foot_lower}" upper="${foot_upper}" />
     <parent link="LD_link"/>
     <child link="LF_link"/>
@@ -198,10 +179,10 @@
   <link name="LF_link">
     <gazebo>
-        <self_collide>1</self_collide>
+      <self_collide>1</self_collide>
     </gazebo>
     <collision>
       <origin xyz="${foot_length/2-down_width/2} ${-foot_width/2} ${-foot_height/2}" rpy="0 0 0"/>
       <geometry>
-	    <box size="${foot_length} ${foot_width} ${foot_height}"/>
+        <box size="${foot_length} ${foot_width} ${foot_height}"/>
       </geometry>
     </collision>
@@ -209,5 +190,5 @@
       <origin xyz="${foot_length/2-down_width/2} ${-foot_width/2} ${-foot_height/2}" rpy="0 0 0"/>
       <geometry>
-	    <box size="${foot_length} ${foot_width} ${foot_height}"/>
+        <box size="${foot_length} ${foot_width} ${foot_height}"/>
       </geometry>
       <material name="orange"/>
@@ -216,13 +197,9 @@
       <origin xyz="${foot_length/2-down_width/2} ${-foot_width/2} ${-foot_height/2}" rpy="0 0 0"/>
       <mass value="${foot_mass}"/>
-      <inertia
-	  ixx="${foot_mass / 12.0 * (foot_width*foot_width + foot_height*foot_height)}" ixy="0.0" ixz="0.0"
-	  iyy="${foot_mass / 12.0 * (foot_length*foot_length + foot_height*foot_height)}" iyz="0.0"
-	  izz="${foot_mass / 12.0 * (foot_length*foot_length + foot_width*foot_width)}"/>
+      <inertia ixx="${foot_mass / 12.0 * (foot_width*foot_width + foot_height*foot_height)}" ixy="0.0" ixz="0.0" iyy="${foot_mass / 12.0 * (foot_length*foot_length + foot_height*foot_height)}" iyz="0.0" izz="${foot_mass / 12.0 * (foot_length*foot_length + foot_width*foot_width)}"/>
     </inertial>
   </link>
   <joint name="RF_joint" type="revolute">
-    <limit
-       velocity="${foot_maxvel}" effort="${foot_effort}" lower="${foot_lower}" upper="${foot_upper}" />
+    <limit velocity="${foot_maxvel}" effort="${foot_effort}" lower="${foot_lower}" upper="${foot_upper}" />
     <parent link="RD_link"/>
     <child link="RF_link"/>
@@ -235,5 +212,5 @@
       <origin xyz="${foot_length/2-down_width/2} ${foot_width/2} ${-foot_height/2}" rpy="0 0 0"/>
       <geometry>
-	    <box size="${foot_length} ${foot_width} ${foot_height}"/>
+        <box size="${foot_length} ${foot_width} ${foot_height}"/>
       </geometry>
     </collision>
@@ -241,5 +218,5 @@
       <origin xyz="${foot_length/2-down_width/2} ${foot_width/2} ${-foot_height/2}" rpy="0 0 0"/>
       <geometry>
-	    <box size="${foot_length} ${foot_width} ${foot_height}"/>
+        <box size="${foot_length} ${foot_width} ${foot_height}"/>
       </geometry>
       <material name="orange"/>
@@ -248,8 +225,5 @@
       <origin xyz="${foot_length/2-down_width/2} ${foot_width/2} ${-foot_height/2}" rpy="0 0 0"/>
       <mass value="${foot_mass}"/>
-      <inertia
-	  ixx="${foot_mass / 12.0 * (foot_width*foot_width + foot_height*foot_height)}" ixy="0.0" ixz="0.0"
-	  iyy="${foot_mass / 12.0 * (foot_length*foot_length + foot_height*foot_height)}" iyz="0.0"
-	  izz="${foot_mass / 12.0 * (foot_length*foot_length + foot_width*foot_width)}"/>
+      <inertia ixx="${foot_mass / 12.0 * (foot_width*foot_width + foot_height*foot_height)}" ixy="0.0" ixz="0.0" iyy="${foot_mass / 12.0 * (foot_length*foot_length + foot_height*foot_height)}" iyz="0.0" izz="${foot_mass / 12.0 * (foot_length*foot_length + foot_width*foot_width)}"/>
     </inertial>
   </link>
